File: RevampDrone/Radio.kicad_sch (KiCad schematic)
At the start: 1 part, among them U12 NRF24L01

Commit message: Get it on V7
Changed lines of the file:
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@@
 (kicad_sch (version 20230121) (generator eeschema)
   (paper "A4")
-  (symbol (lib_id "RF:NRF24L01") (at 142.875 91.44 0) (unit 1)
+  (symbol (lib_id "RF:NRF24L01") (at 141.605 97.79 0) (unit 1)
     (in_bom yes) (on_board yes) (dnp no) (fields_autoplaced)
-    (property "Reference" "U12" (at 147.3709 71.12 0)
+    (property "Reference" "U12" (at 146.1009 77.47 0)
       (effects (font (size 1.27 1.27)) (justify left))
     )
-    (property "Value" "NRF24L01" (at 147.3709 73.66 0)
+    (property "Value" "NRF24L01" (at 146.1009 80.01 0)
       (effects (font (size 1.27 1.27)) (justify left))
     )
-    (property "Footprint" "Package_DFN_QFN:QFN-20-1EP_4x4mm_P0.5mm_EP2.5x2.5mm" (at 147.955 71.12 0)
+    (property "Footprint" "Package_DFN_QFN:QFN-20-1EP_4x4mm_P0.5mm_EP2.5x2.5mm" (at 146.685 77.47 0)
       (effects (font (size 1.27 1.27) italic) (justify left) hide)
     )
-    (property "Datasheet" "http://www.nordicsemi.com/eng/content/download/2730/34105/file/nRF24L01_Product_Specification_v2_0.pdf" (at 142.875 88.9 0)
+    (property "Datasheet" "http://www.nordicsemi.com/eng/content/download/2730/34105/file/nRF24L01_Product_Specification_v2_0.pdf" (at 141.605 95.25 0)
       (effects (font (size 1.27 1.27)) hide)
     )
@@
     (pin "9")
     (instances
-      (project "DroneRevamp"
-        (path "/b197cc17-7ac5-409f-9705-26347f5a482b/2c964ca4-8801-4c94-a547-fc606af1506f"
+      (project "RevampDrone"
+        (path "/a57dd8a7-b3ae-4be1-9fc6-9c9c7e0e2ba9/0bc43be2-7c83-4054-ab5e-b7ae25f9fc7a"
           (reference "U12") (unit 1)
         )
